File: kicad/flight-controller/esp32s3.kicad_sch (KiCad schematic)
At the start: 15 parts, among them J13 USB_C_Receptacle_USB2.0_16P, SW1 TS-1088, SW2 TS-1088, U1 ESP32-S3-WROOM-1

Commit message: Fix ESP32 LDO thermal margin, add USB-C/SBUS ESD protection
Design review flagged the ESP32-S3's 3.3V LDO (AP2112K-3.3, SOT-23-5)
at only 1.5C margin to absolute max under WiFi load. Swapped to a
Torex XC6220B331PR-G (SOT-89-5, thermal tab tied to GND) with matching
input/output caps and thermal vias under the tab; thermal score is now
100/100 with no findings. Sensor LDO (U6) was unaffected and left as-is.

Also added TVS protection that was missing on two exposed signal paths:
D4 + bulk cap on USB-C VBUS (J13, now populated for field use) ahead of
the existing blocking diode, and a matching TVS (D6) on the RC receiver
SBUS line (J7), reusing the same part to minimize BOM diversity.

Every part number touched this pass (U4, C17-C19, D4, D6) was verified
against real distributor data, and a full BOM audit confirmed all other
assigned part numbers match their stated value and footprint. Also
removed two orphaned, unwired schematic files (airspeed.kicad_sch,
lidar.kicad_sch) that weren't in the sheet hierarchy.

Known follow-up before fab: the production/ fab package predates this
rework and needs to be regenerated, and Update PCB from Schematic needs
a re-run to sync D4/D6's display value (nets are already correct).

Co-Authored-By: Claude Sonnet 5 <noreply@anthropic.com>
Claude-Session: https://claude.ai/code/session_01NksRnW4jXLWsYwZNR7u39H
Parts:
- C17: LCSC Part (none) -> C440198; Notes USB VBUS bulk/decoupling cap (added in review) - value/volt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 -> USB VBUS bulk/decoupling cap (added in review)
- D4: value TVS 5V -> ESD5Z5.0T1G; LCSC Part (none) -> C82044; Notes USB VBUS ESD/surge protection (added in review) - specific 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 -> USB VBUS ESD/surge protection (added in review)
- J13: value USB_C_Receptacle_USB2.0_16P -> USB-C
- SW1: Notes Reset button -> Reset
- SW2: Notes Boot button -> Boot
Changed lines of the file:
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@@
 		(title "ESP32")
 		(date "2026-09-09")
-		(rev "v3.0")
+		(rev "v3.1")
 		(company "Travis Brown")
 		(comment 1 "ESP32-S3-N16-R8 Wroom 1 Module")
@@
 			)
 		)
-		(property "Value" "USB_C_Receptacle_USB2.0_16P"
+		(property "Value" "USB-C"
 			(at 200.914 145.034 90)
 			(show_name no)
@@
 			)
 		)
-		(property "Value" "TVS 5V"
+		(property "Value" "ESD5Z5.0T1G"
 			(at 138.43 125.38 0)
 			(show_name no)
@@
 			)
 		)
-		(property "Datasheet" ""
+		(property "Datasheet" "https://www.lcsc.com/datasheet/C82044.pdf"
 			(at 138.43 118.11 0)
 			(hide yes)
@@
 			)
 		)
-		(property "Description" "TVS diode"
+		(property "Description" "TVS diode, onsemi, 5V standoff / 6.2V breakdown, unidirectional"
 			(at 138.43 118.11 0)
 			(hide yes)
@@
 			)
 		)
-		(property "Notes" "USB VBUS ESD/surge protection (added in review) - specific MPN not yet sourced, select a 5V-rated USB VBUS TVS before BOM lock"
+		(property "Notes" "USB VBUS ESD/surge protection (added in review)"
+			(at 138.43 118.11 0)
+			(hide yes)
+			(show_name no)
+			(do_not_autoplace no)
+			(effects
+				(font
+					(size 1.27 1.27)
+				)
+			)
+		)
+		(property "LCSC Part" "C82044"
 			(at 138.43 118.11 0)
 			(hide yes)
@@
 			)
 		)
-		(property "Notes" "Boot button"
+		(property "Notes" "Boot"
 			(at 262.89 144.78 0)
 			(hide yes)
@@
 			)
 		)
-		(property "Notes" "Reset button"
+		(property "Notes" "Reset"
 			(at 247.65 116.84 0)
 			(hide yes)
@@
 			)
 		)
-		(property "Datasheet" ""
+		(property "Datasheet" "https://www.lcsc.com/datasheet/C440198.pdf"
 			(at 154.94 128.27 0)
 			(hide yes)
@@
 			)
 		)
-		(property "Description" "Unpolarized capacitor"
+		(property "Description" "Unpolarized capacitor, Murata GRM21BR61H106KE43L, 50V X5R"
 			(at 154.94 128.27 0)
 			(hide yes)
@@
 			)
 		)
-		(property "Notes" "USB VBUS bulk/decoupling cap (added in review) - value/voltage rating not yet sourced"
+		(property "Notes" "USB VBUS bulk/decoupling cap (added in review)"
 			(at 154.94 128.27 0)
 			(hide yes)
+			(show_name no)
+			(do_not_autoplace no)
+			(effects
+				(font
+					(size 1.27 1.27)
+				)
+			)
+		)
+		(property "LCSC Part" "C440198"
+			(at 154.94 128.27 0)
+			(hide yes)
