File: kicad/flight-controller/servo_out.kicad_sch (KiCad schematic)
At the start: 16 parts, among them J1 1, J16 8, J2 2, J3 3, J4 4, J5 5, J6 6, J9 7

Commit message: removed basestation code and v3.1 of fc pcb
Parts:
- removed J16: 8, Connector_Molex:Molex_KK-254_AE-6410-03A_1x03_P2.54mm_Vertical, symbol Connector:Conn_01x03_Pin
- removed J9: 7, Connector_Molex:Molex_KK-254_AE-6410-03A_1x03_P2.54mm_Vertical, symbol Connector:Conn_01x03_Pin
- removed R16, R17: 330R, Resistor_SMD:R_0402_1005Metric, symbol Device:R
Connections:
- net SERVO_OUT_4: now also R19.1; no longer R15.1
- net SERVO_OUT_5: now also R18.1; no longer R19.1
- net SERVO_OUT_6: now also R15.1; no longer R18.1
- net at J4.1 (Pin_1): now also R19.2; no longer R15.2
- net at J6.1 (Pin_1): now also R15.2; no longer R18.2
- net at J5.1 (Pin_1): now also R18.2; no longer R19.2
Other:
- note removed: "Extra Output 1"
- note removed: "Extra Output 2"
