File: kicad/flight-controller/fc_ldo.kicad_sch (KiCad schematic)
At the start: 6 parts, among them U4 XC6220B331PR-G, U6 AP2112K-3.3

Commit message: removed basestation code and v3.1 of fc pcb
Parts:
- added TP10: GND, TestPoint:TestPoint_THTPad_D1.0mm_Drill0.5mm, symbol Connector:TestPoint
- added TP7: ESP_3V3, TestPoint:TestPoint_Pad_D1.0mm, symbol Connector:TestPoint
- added TP8: SENSOR_3V3, TestPoint:TestPoint_Pad_D1.0mm, symbol Connector:TestPoint
- added TP9: FC_5V, TestPoint:TestPoint_THTPad_D1.5mm_Drill0.7mm, symbol Connector:TestPoint
Connections:
- net ESP_3V3: now also TP7.1
- net FC_5V: now also TP9.1
- net GND: now also TP10.1
- net SENSOR_3V3: now also TP8.1

Commit message: Kicad FC v3.1 complete, Mission Controller and UWB boards v1 complete, firmware v2 complete!
Parts:
- C18: value 10uF -> 22uF; footprint Capacitor_SMD:C_0603_1608Metric -> Capacitor_SMD:C_0805_2012Metric; LCSC Part C1691 -> C45783
- TP10, TP7, TP8, TP9: now left out of the parts list
Changed lines of the file:
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@@
 		(body_style 1)
 		(exclude_from_sim no)
-		(in_bom yes)
-		(on_board yes)
-		(in_pos_files yes)
+		(in_bom no)
+		(on_board yes)
+		(in_pos_files no)
 		(dnp no)
 		(property "Reference" "TP10"
@@
 			)
 		)
-		(property "Value" "10uF"
+		(property "Value" "22uF"
 			(at 159.004 94.234 0)
 			(show_name no)
@@
 			)
 		)
-		(property "Footprint" "Capacitor_SMD:C_0603_1608Metric"
+		(property "Footprint" "Capacitor_SMD:C_0805_2012Metric"
 			(at 160.3248 91.44 0)
 			(hide yes)
@@
 			)
 		)
-		(property "LCSC Part" "C1691"
+		(property "LCSC Part" "C45783"
 			(at 161.29 95.25 0)
 			(hide yes)
@@
 		(body_style 1)
 		(exclude_from_sim no)
-		(in_bom yes)
-		(on_board yes)
-		(in_pos_files yes)
+		(in_bom no)
+		(on_board yes)
+		(in_pos_files no)
 		(dnp no)
 		(property "Reference" "TP8"
@@
 		(body_style 1)
 		(exclude_from_sim no)
-		(in_bom yes)
-		(on_board yes)
-		(in_pos_files yes)
+		(in_bom no)
+		(on_board yes)
+		(in_pos_files no)
 		(dnp no)
 		(property "Reference" "TP7"
@@
 		(body_style 1)
 		(exclude_from_sim no)
-		(in_bom yes)
-		(on_board yes)
-		(in_pos_files yes)
+		(in_bom no)
+		(on_board yes)
+		(in_pos_files no)
 		(dnp no)
 		(property "Reference" "TP9"
