File: kicad/flight-controller/microsd.kicad_sch (KiCad schematic)
At the start: 5 parts

Commit message: removed basestation code and v3.1 of fc pcb
Connections:
- net ESP_3V3: now also C13.2, Card1.4 (VDD); no longer C13.1
- net GND: now also C13.1
Changed lines of the file:
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@@
+	)
+	(junction
+		(at 129.54 91.44)
+		(diameter 0)
+		(color 0 0 0 0)
 	)
 	(junction
@@
 		(pts
 			(xy 129.54 91.44) (xy 142.24 91.44)
+		)
+		(stroke
+			(width 0)
+			(type default)
+		)
+	)
+	(wire
+		(pts
+			(xy 129.54 91.44) (xy 121.92 91.44)
 		)
 		(stroke
@@
 	(hierarchical_label "ESP_3V3"
 		(shape input)
-		(at 129.54 83.82 180)
+		(at 121.92 91.44 180)
 		(effects
 			(font
@@
 		(effects
 			(font
+				(size 1.27 1.27)
+			)
+			(justify right)
+		)
+	)
+	(hierarchical_label "GND"
+		(shape input)
+		(at 129.54 83.82 180)
+		(effects
+			(font

Commit message: Kicad FC v3.1 complete, Mission Controller and UWB boards v1 complete, firmware v2 complete!
Parts:
- added R28, R29, R30: 10K, Resistor_SMD:R_0402_1005Metric, symbol Device:R
Connections:
- net ESP_3V3: now also R28.2, R29.2, R30.2
- net MISO: now also R28.1
- net MOSI: now also R30.1
- net SD_CS: now also R29.1
Other:
- moved on the sheet: R11, R2
