File: kicad/mission-board/camera.kicad_sch (KiCad schematic)
At the start: 3 parts, among them J13 Camera FPC, U10 24MHz Oscillator

Commit message: pcb progress
Other:
- moved on the sheet: C6

Commit message: progress on v1 of mission board
Parts:
- added C25, C26, C27, C28: 1uF, Capacitor_SMD:C_0402_1005Metric, symbol Device:C
- added R37, R38: 10k, Resistor_SMD:R_0402_1005Metric, symbol Device:R
- added U16: XC6206P282MR, Package_TO_SOT_SMD:SOT-23-3, symbol Regulator_Linear:XC6206PxxxMR
- added U17: XC6206P122MR, Package_TO_SOT_SMD:SOT-23-3, symbol Regulator_Linear:XC6206PxxxMR
Connections:
- net CAM_D0: now also J13.6; no longer J13.1
- net CAM_D1: now also J13.4; no longer J13.2
- net CAM_D3: now also J13.5; no longer J13.4
- net CAM_D4: now also J13.7; no longer J13.5
- net CAM_D5: now also J13.9; no longer J13.6
- net CAM_D6: now also J13.11; no longer J13.7
- net CAM_D7: now also J13.13; no longer J13.8
- net CAM_HREF: now also J13.16; no longer J13.11
- net CAM_PCLK: now also J13.8; no longer J13.9
- net CAM_PWDN: now also J13.17, R37.2; no longer J13.15
- net CAM_RESET: now also J13.19, R38.2; no longer J13.16
- net CAM_VSYNC: now also J13.18; no longer J13.10
- net ESP_3V3: now also J13.14, U10.1 (Tri-state), C25.1, C27.1, R37.1, R38.1, U16.3 (VI), U17.3 (VI); no longer J13.18
- net GND: now also J13.10, J13.23, C25.2, C26.2, C27.2, C28.2, U16.1 (GND), U17.1 (GND); no longer J13.17
- net I2C_SCL: now also J13.20; no longer J13.13
- net I2C_SDA: now also J13.22; no longer J13.14
- net CAM_2V8: now reaches J13.21
- net CAM_2V8: now also C26.1, U16.2 (VO)
- new net CAM_1V2: C28.1, J13.15, U17.2 (VO)
- no-connect marks 7 -> 3
Other:
- moved on the sheet: U10

Commit message: Kicad FC v3.1 complete, Mission Controller and UWB boards v1 complete, firmware v2 complete!
Other:
- note removed: "PLACEHOLDER PINOUT: verify against the exact camera module datasheet before fab."
Changed lines of the file:
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@@
 		(rev "v1.0")
-	)
-	(text "PLACEHOLDER PINOUT: verify against the exact camera module datasheet before fab."
-		(exclude_from_sim no)
-		(at 69.088 34.798 0)
-		(effects
-			(font
-				(size 1.27 1.27)
-			)
-		)
 	)
 	(no_connect
@@
 		(dnp no)
 		(property "Reference" "C25"
-			(at 134.62 49.53 0)
+			(at 120.396 49.53 0)
 			(show_name no)
 			(do_not_autoplace no)
@@
 		)
 		(property "Value" "1uF"
-			(at 134.62 52.07 0)
+			(at 120.396 52.07 0)
 			(show_name no)
 			(do_not_autoplace no)
@@
 		(dnp no)
 		(property "Reference" "U17"
-			(at 154.94 87.63 0)
+			(at 149.352 84.582 0)
 			(show_name no)
 			(do_not_autoplace no)
@@
 		)
 		(property "Value" "XC6206P122MR"
-			(at 154.94 90.17 0)
+			(at 145.034 82.296 0)
 			(show_name no)
 			(do_not_autoplace no)
@@
 		(dnp no)
 		(property "Reference" "C27"
-			(at 134.62 87.63 0)
+			(at 124.714 86.868 0)
 			(show_name no)
 			(do_not_autoplace no)
@@
 		)
 		(property "Value" "1uF"
-			(at 134.62 90.17 0)
+			(at 124.714 89.408 0)
 			(show_name no)
 			(do_not_autoplace no)
@@
 		(dnp no)
 		(property "Reference" "U16"
-			(at 154.94 49.53 0)
+			(at 149.86 66.548 0)
 			(show_name no)
 			(do_not_autoplace no)
@@
 		)
 		(property "Value" "XC6206P282MR"
-			(at 154.94 52.07 0)
-			(show_name no)
-			(do_not_autoplace no)
+			(at 144.272 64.262 0)
+			(show_name no)
+			(do_not_autoplace no)
