File: kicad/mission-board/esp32_core.kicad_sch (KiCad schematic)
At the start: 11 parts, among them J21 Fast IO Expansion, SW1 TS-1088, SW2 TS-1088, U11 ESP32-S3-WROOM-1

Commit message: pcb progress
Parts:
- J21: footprint Connector_PinHeader_2.54mm:PinHeader_1x06_P2.54mm_Vertical -> Connector_PinHeader_2.54mm:PinHeader_1x05_P2.54mm_Vertical
Changed lines of the file:
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@@
 		)
 		(property "Value" "Fast IO Expansion"
-			(at 214.92 147.62 0)
+			(at 208.788 139.7 0)
 			(show_name no)
 			(do_not_autoplace no)
@@
 			)
 		)
-		(property "Footprint" "Connector_PinHeader_2.54mm:PinHeader_1x06_P2.54mm_Vertical"
+		(property "Footprint" "Connector_PinHeader_2.54mm:PinHeader_1x05_P2.54mm_Vertical"
 			(at 220 140 0)
 			(hide yes)

Commit message: progress on v1 of mission board
Parts:
- C7: value 100nF -> 1uF; LCSC Part C1525 -> C52923
- J21: symbol Connector:Conn_01x06_Pin -> Connector:Conn_01x05_Pin
Connections:
- net CAM_D0: now also U11.25 (IO48); no longer U11.26 (IO45)
- net CAM_D1: now also U11.23 (IO21); no longer U11.24 (IO47)
- net CAM_D2: now also U11.22 (IO14); no longer U11.25 (IO48)
- net CAM_D3: now also U11.24 (IO47); no longer U11.38 (IO2)
- net CAM_D4: now also U11.31 (IO38); no longer U11.12 (IO8)
- net CAM_D5: now also U11.33 (IO40); no longer U11.17 (IO9)
- net CAM_D6: now also U11.34 (IO41); no longer U11.18 (IO10)
- net CAM_D7: now also U11.35 (IO42); no longer U11.19 (IO11)
- net CAM_HREF: now also U11.8 (IO15); no longer U11.35 (IO42)
- net CAM_PCLK: now also U11.32 (IO39); no longer U11.33 (IO40)
- net CAM_VSYNC: now also U11.7 (IO7); no longer U11.34 (IO41)
- net FASTIO1: now also U11.39 (IO1); no longer U11.5 (IO5)
- net FASTIO2: now also U11.38 (IO2); no longer U11.6 (IO6)
- net FASTIO3: now also U11.15 (IO3); no longer U11.7 (IO7)
- net HBRIDGE_AIN1: now also U11.4 (IO4); no longer U11.20 (IO12)
- net HBRIDGE_AIN2: now also U11.5 (IO5); no longer U11.21 (IO13)
- net HBRIDGE_BIN1: now also U11.6 (IO6); no longer U11.22 (IO14)
- net HBRIDGE_BIN2: now also U11.26 (IO45); no longer U11.8 (IO15)
- net I2C_SDA: now also U11.12 (IO8); no longer U11.10 (IO17)
- net INTER_ESP_UART_RX: now also U11.20 (IO12); no longer U11.15 (IO3)
- net INTER_ESP_UART_TX: now also U11.21 (IO13); no longer U11.9 (IO16)
- net LED_NODE: no longer D9.2 (A), R28.2
- net MCP_INT: now also U11.9 (IO16); no longer U11.4 (IO4)
- net SENSE_MUX_OUT: now also U11.10 (IO17); no longer U11.39 (IO1)
- net SPI_MISO: now also U11.18 (IO10); no longer U11.31 (IO38)
- net SPI_MOSI: now also U11.19 (IO11); no longer U11.23 (IO21)
- net SPI_SCK: now also U11.17 (IO9); no longer U11.32 (IO39)
- new net LED_A: D9.2 (A), R28.2
Changed lines of the file:
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@@
 	)
 	(label "FASTIO3"
-		(at 105.41 130.81 180)
+		(at 114.3 162.56 270)
 		(effects
 			(font
@@
 	)
 	(label "FASTIO2"
-		(at 105.41 128.27 180)
-		(effects
-			(font
-				(size 1.27 1.27)
-			)
-			(justify right)
+		(at 148.59 120.65 0)
+		(effects
+			(font
+				(size 1.27 1.27)
+			)
+			(justify left)
 		)
 	)
@@
 		)
 	)
-	(label "LED_NODE"
+	(label "LED_A"
 		(at 34.29 167.64 0)
 		(effects
@@
 		)
 	)
-	(label "LED_NODE"
+	(label "LED_A"
 		(at 59.69 158.75 0)
 		(effects
@@
 	)
 	(label "FASTIO1"
-		(at 105.41 125.73 180)
-		(effects
-			(font
-				(size 1.27 1.27)
-			)
-			(justify right)
+		(at 148.59 118.11 0)
+		(effects
+			(font
+				(size 1.27 1.27)
+			)
+			(justify left)
 		)
 	)
@@
 	(hierarchical_label "HBRIDGE_BIN2"
 		(shape output)
-		(at 105.41 133.35 180)
+		(at 142.24 162.56 270)
 		(effects
 			(font
@@
 	(hierarchical_label "SPI_SCK"
 		(shape output)
-		(at 148.59 135.89 0)
-		(effects
-			(font
-				(size 1.27 1.27)
-			)
-			(justify left)
+		(at 119.38 162.56 270)
+		(effects
+			(font
+				(size 1.27 1.27)
+			)
+			(justify right)
 		)
 	)
@@
 	(hierarchical_label "SPI_MISO"
 		(shape input)
-		(at 148.59 138.43 0)
-		(effects
-			(font
-				(size 1.27 1.27)
-			)
-			(justify left)
+		(at 121.92 162.56 270)
+		(effects
+			(font
+				(size 1.27 1.27)
+			)
+			(justify right)
 		)
 	)
 	(hierarchical_label "INTER_ESP_UART_TX"
 		(shape output)
-		(at 105.41 135.89 180)
+		(at 129.54 162.56 270)
 		(effects
 			(font
@@
 	(hierarchical_label "SPI_MOSI"
 		(shape output)
-		(at 134.62 162.56 270)
+		(at 124.46 162.56 270)
 		(effects
 			(font
@@
 	(hierarchical_label "HBRIDGE_AIN1"
 		(shape output)
-		(at 127 162.56 270)
+		(at 105.41 123.19 180)
 		(effects
 			(font
@@
 	(hierarchical_label "CAM_D4"
 		(shape input)
-		(at 105.41 143.51 180)
-		(effects
-			(font
-				(size 1.27 1.27)
-			)
-			(justify right)
+		(at 148.59 138.43 0)
+		(effects
+			(font
+				(size 1.27 1.27)
+			)
+			(justify left)
 		)
 	)
 	(hierarchical_label "CAM_D1"
 		(shape input)
-		(at 137.16 162.56 270)
+		(at 134.62 162.56 270)
 		(effects
 			(font
@@
 	(hierarchical_label "HBRIDGE_AIN2"
 		(shape output)
-		(at 129.54 162.56 270)
+		(at 105.41 125.73 180)
 		(effects
 			(font
@@
 	(hierarchical_label "CAM_PCLK"
 		(shape input)
+		(at 148.59 135.89 0)
+		(effects
+			(font
+				(size 1.27 1.27)
+			)
+			(justify left)
+		)
+	)
+	(hierarchical_label "CAM_D2"
+		(shape input)
+		(at 132.08 162.56 270)
+		(effects
+			(font
+				(size 1.27 1.27)
+			)
+			(justify right)
+		)
+	)
+	(hierarchical_label "DEBUG_UART_RX"
+		(shape input)
+		(at 148.59 125.73 0)
+		(effects
+			(font
+				(size 1.27 1.27)
+			)
+			(justify left)
+		)
+	)
+	(hierarchical_label "INTER_ESP_UART_RX"
+		(shape input)
+		(at 127 162.56 270)
+		(effects
+			(font
+				(size 1.27 1.27)
+			)
+			(justify right)
+		)
+	)
+	(hierarchical_label "CAM_D3"
+		(shape input)
+		(at 137.16 162.56 270)
+		(effects
+			(font
+				(size 1.27 1.27)
+			)
+			(justify right)
+		)
+	)
+	(hierarchical_label "MCP_INT"
+		(shape input)
+		(at 105.41 135.89 180)
+		(effects
+			(font
+				(size 1.27 1.27)
+			)
+			(justify right)
+		)
+	)
+	(hierarchical_label "CAM_D7"
+		(shape input)
+		(at 148.59 128.27 0)
+		(effects
+			(font
+				(size 1.27 1.27)
+			)
+			(justify left)
+		)
+	)
+	(hierarchical_label "CAM_VSYNC"
+		(shape input)
+		(at 105.41 130.81 180)
+		(effects
+			(font
+				(size 1.27 1.27)
+			)
+			(justify right)
+		)
+	)
+	(hierarchical_label "CAM_D5"
+		(shape input)
 		(at 148.59 133.35 0)
 		(effects
@@
 			)
 			(justify left)
-		)
-	)
-	(hierarchical_label "CAM_D2"
-		(shape input)
-		(at 139.7 162.56 270)
-		(effects
-			(font
-				(size 1.27 1.27)
-			)
-			(justify right)
-		)
-	)
-	(hierarchical_label "DEBUG_UART_RX"
-		(shape input)
-		(at 148.59 125.73 0)
-		(effects
-			(font
-				(size 1.27 1.27)
-			)
-			(justify left)
-		)
-	)
-	(hierarchical_label "INTER_ESP_UART_RX"
-		(shape input)
-		(at 114.3 162.56 270)
-		(effects
-			(font
-				(size 1.27 1.27)
-			)
-			(justify right)
-		)
-	)
-	(hierarchical_label "CAM_D3"
-		(shape input)
-		(at 148.59 120.65 0)
-		(effects
-			(font
-				(size 1.27 1.27)
-			)
-			(justify left)
-		)
-	)
-	(hierarchical_label "MCP_INT"
-		(shape input)
-		(at 105.41 123.19 180)
-		(effects
-			(font
-				(size 1.27 1.27)
-			)
-			(justify right)
-		)
-	)
-	(hierarchical_label "CAM_D7"
-		(shape input)
-		(at 124.46 162.56 270)
-		(effects
-			(font
-				(size 1.27 1.27)
-			)
-			(justify right)
-		)
-	)
-	(hierarchical_label "CAM_VSYNC"
-		(shape input)
-		(at 148.59 130.81 0)
-		(effects
-			(font
-				(size 1.27 1.27)
-			)
-			(justify left)
-		)
-	)
-	(hierarchical_label "CAM_D5"
-		(shape input)
-		(at 119.38 162.56 270)
-		(effects
-			(font
-				(size 1.27 1.27)
-			)
-			(justify right)
 		)
 	)
 	(hierarchical_label "I2C_SDA"
 		(shape bidirectional)
-		(at 105.41 138.43 180)
+		(at 105.41 143.51 180)
 		(effects
 			(font
@@
 	(hierarchical_label "CAM_D6"
 		(shape input)
-		(at 121.92 162.56 270)
-		(effects
-			(font
-				(size 1.27 1.27)
-			)
-			(justify right)
+		(at 148.59 130.81 0)
+		(effects
+			(font
+				(size 1.27 1.27)
+			)
+			(justify left)
 		)
 	)
 	(hierarchical_label "CAM_D0"
 		(shape input)
-		(at 142.24 162.56 270)
+		(at 139.7 162.56 270)
 		(effects
 			(font
@@
 	(hierarchical_label "HBRIDGE_BIN1"
 		(shape output)
-		(at 132.08 162.56 270)
+		(at 105.41 128.27 180)
 		(effects
 			(font
@@
 	(hierarchical_label "SENSE_MUX_OUT"
 		(shape input)
-		(at 148.59 118.11 0)
-		(effects
-			(font
-				(size 1.27 1.27)
-			)
-			(justify left)
+		(at 105.41 138.43 180)
+		(effects
+			(font
+				(size 1.27 1.27)
+			)
+			(justify right)
 		)
 	)
 	(hierarchical_label "CAM_HREF"
 		(shape input)
-		(at 148.59 128.27 0)
-		(effects
-			(font
-				(size 1.27 1.27)
-			)
-			(justify left)
+		(at 105.41 133.35 180)
+		(effects
+			(font
+				(size 1.27 1.27)
+			)
+			(justify right)
 		)
 	)
@@
 	)
 	(symbol
-		(lib_id "Connector:Conn_01x06_Pin")
+		(lib_id "Connector:Conn_01x05_Pin")
 		(at 220 140 0)
 		(unit 1)
@@
 		)
 		(pin "5"
-		)
-		(pin "6"
 		)
 		(instances
@@
 			)
 		)
-		(property "Value" "100nF"
+		(property "Value" "1uF"
 			(at 40.64 55.88 0)
 			(show_name no)
@@
 			)
 		)
-		(property "Description" ""
+		(property "Description" "ESP32 EN RC delay (10k/1uF per Espressif HW guidelines)"
 			(at 45.72 53.34 0)
 			(show_name no)
@@
 			)
 		)
-		(property "LCSC Part" "C1525"
+		(property "LCSC Part" "C52923"
 			(at 45.72 53.34 0)
 			(hide yes)

Commit message: Kicad FC v3.1 complete, Mission Controller and UWB boards v1 complete, firmware v2 complete!
Parts:
- C9: value 10uF -> 22uF
- D9: LCSC Part C2289 -> C2286
- J21: LCSC Part (none) -> C2895846
- R26, R27: LCSC Part C25531 -> C25744
Connections:
- net CAM_D0: now also U11.22 (IO14); no longer U11.25 (IO48)
- net CAM_D1: now also U11.24 (IO47); no longer U11.23 (IO21)
- net CAM_D2: now also U11.25 (IO48); no longer U11.22 (IO14)
- net CAM_D3: now also U11.23 (IO21); no longer U11.24 (IO47)
- net INTER_ESP_UART_RX: now also U11.21 (IO13); no longer U11.20 (IO12)
- net INTER_ESP_UART_TX: now also U11.20 (IO12); no longer U11.21 (IO13)
- net SPI_MISO renamed FASTIO5
- net SPI_MOSI: no longer names the net of U11.19 (IO11)
- net SPI_SCK renamed FASTIO4
- no-connect marks 3 -> 4
Changed lines of the file:
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@@
+	)
+	(no_connect
+		(at 124.46 162.56)
 	)
 	(no_connect
@@
 	(wire
 		(pts
-			(xy 225.08 137.46) (xy 230.16 137.46)
-		)
-		(stroke
-			(width 0)
-			(type default)
-		)
-	)
-	(wire
-		(pts
 			(xy 177.8 110.49) (xy 177.8 105.41)
 		)
@@
 	(wire
 		(pts
-			(xy 225.08 134.92) (xy 230.16 134.92)
-		)
-		(stroke
-			(width 0)
-			(type default)
-		)
-	)
-	(wire
-		(pts
 			(xy 52.07 35.56) (xy 46.99 35.56)
 		)
@@
 	(wire
 		(pts
-			(xy 225.08 145.08) (xy 230.16 145.08)
+			(xy 224.79 144.78) (xy 231.14 144.78)
+		)
+		(stroke
+			(width 0)
+			(type default)
+		)
+	)
+	(wire
+		(pts
+			(xy 224.79 137.16) (xy 231.14 137.16)
 		)
 		(stroke
@@
 	(wire
 		(pts
+			(xy 224.79 139.7) (xy 231.14 139.7)
+		)
+		(stroke
+			(width 0)
+			(type default)
+		)
+	)
+	(wire
+		(pts
 			(xy 54.61 158.75) (xy 59.69 158.75)
 		)
@@
 	(wire
 		(pts
-			(xy 225.08 142.54) (xy 230.16 142.54)
+			(xy 224.79 142.24) (xy 231.14 142.24)
 		)
 		(stroke
@@
 	(wire
 		(pts
-			(xy 225.08 140) (xy 230.16 140)
-		)
-		(stroke
-			(width 0)
-			(type default)
-		)
-	)
-	(wire
-		(pts
 			(xy 33.02 107.95) (xy 33.02 113.03)
+		)
+		(stroke
+			(width 0)
+			(type default)
+		)
+	)
+	(wire
+		(pts
+			(xy 224.79 134.62) (xy 231.14 134.62)
 		)
 		(stroke
@@
 	)
 	(label "FASTIO1"
-		(at 230.16 140 0)
+		(at 231.14 139.7 0)
 		(effects
 			(font
@@
 	)
 	(label "FASTIO2"
-		(at 230.16 142.54 0)
+		(at 231.14 142.24 0)
 		(effects
 			(font
@@
 	)
 	(label "FASTIO3"
-		(at 230.16 145.08 0)
+		(at 231.14 144.78 0)
 		(effects
 			(font
@@
 	)
 	(label "ESP_3V3"
-		(at 230.16 134.92 0)
+		(at 231.14 134.62 0)
 		(effects
 			(font
@@
 	)
 	(label "GND"
-		(at 230.16 137.46 0)
+		(at 231.14 137.16 0)
 		(effects
 			(font
@@
 		)
 	)
-	(hierarchical_label "SPI_SCK"
-		(shape output)
-		(at 119.38 162.56 270)
-		(effects
-			(font
-				(size 1.27 1.27)
-			)
-			(justify right)
-		)
-	)
 	(hierarchical_label "ESP_3V3"
 		(shape input)
@@
 		)
 	)
+	(hierarchical_label "FASTIO5"
+		(shape bidirectional)
+		(at 121.92 162.56 270)
+		(effects
+			(font
+				(size 1.27 1.27)
+			)
+			(justify right)
+		)
+	)
 	(hierarchical_label "USB_DP"
 		(shape input)
@@
 		)
 	)
-	(hierarchical_label "SPI_MISO"
-		(shape input)
-		(at 121.92 162.56 270)
+	(hierarchical_label "FASTIO4"
+		(shape bidirectional)
+		(at 119.38 162.56 270)
 		(effects
 			(font
@@
 	(hierarchical_label "INTER_ESP_UART_TX"
 		(shape output)
-		(at 129.54 162.56 270)
+		(at 127 162.56 270)
 		(effects
 			(font
@@
 		)
 	)
-	(hierarchical_label "SPI_MOSI"
-		(shape output)
-		(at 124.46 162.56 270)
-		(effects
-			(font
-				(size 1.27 1.27)
-			)
-			(justify right)
-		)
-	)
 	(hierarchical_label "HBRIDGE_AIN1"
 		(shape output)
@@
 	(hierarchical_label "CAM_D1"
 		(shape input)
-		(at 134.62 162.56 270)
+		(at 137.16 162.56 270)
 		(effects
 			(font
@@
 	(hierarchical_label "CAM_D2"
 		(shape input)
-		(at 132.08 162.56 270)
+		(at 139.7 162.56 270)
 		(effects
 			(font
@@
 	(hierarchical_label "INTER_ESP_UART_RX"
 		(shape input)
-		(at 127 162.56 270)
+		(at 129.54 162.56 270)
 		(effects
 			(font
@@
 	(hierarchical_label "CAM_D3"
 		(shape input)
-		(at 137.16 162.56 270)
+		(at 134.62 162.56 270)
 		(effects
 			(font
@@
 	(hierarchical_label "CAM_D0"
 		(shape input)
-		(at 139.7 162.56 270)
+		(at 132.08 162.56 270)
 		(effects
 			(font
@@
 			)
 		)
-		(property "LCSC Part" "C2289"
+		(property "LCSC Part" "C2286"
 			(at 50.8 158.75 0)
 			(hide yes)
@@
 			)
 		)
-		(property "LCSC Part" "C25531"
+		(property "LCSC Part" "C25744"
 			(at 58.42 53.34 0)
 			(hide yes)
@@
 			)
 		)
-		(property "LCSC Part" "C25531"
+		(property "LCSC Part" "C25744"
 			(at 33.02 104.14 0)
 			(hide yes)
@@
 	(symbol
 		(lib_id "Connector:Conn_01x05_Pin")
-		(at 220 140 0)
+		(at 219.71 139.7 0)
 		(unit 1)
 		(body_style 1)
@@
 		(dnp no)
 		(property "Reference" "J21"
-			(at 214.92 132.38 0)
+			(at 214.63 132.08 0)
 			(show_name no)
 			(do_not_autoplace no)
@@
 		)
 		(property "Value" "Fast IO Expansion"
-			(at 208.788 139.7 0)
+			(at 208.498 139.4 0)
 			(show_name no)
 			(do_not_autoplace no)
@@
 		)
 		(property "Footprint" "Connector_PinHeader_2.54mm:PinHeader_1x05_P2.54mm_Vertical"
-			(at 220 140 0)
+			(at 219.71 139.7 0)
 			(hide yes)
 			(show_name no)
@@
 		)
 		(property "Datasheet" ""
-			(at 220 140 0)
+			(at 219.71 139.7 0)
 			(hide yes)
 			(show_name no)
@@
 		)
 		(property "Description" "Direct ESP32-S3 GPIO breakout for future fast/timing-critical IO (IO5-IO7); pin6 not connected"
-			(at 220 140 0)
+			(at 219.71 139.7 0)
+			(hide yes)
+			(show_name no)
+			(do_not_autoplace no)
+			(effects
+				(font
+					(size 1.27 1.27)
+				)
+			)
+		)
+		(property "LCSC Part" "C2895846"
+			(at 219.71 139.7 0)
 			(hide yes)
 			(show_name no)
@@
 			)
 		)
-		(property "Value" "10uF"
+		(property "Value" "22uF"
 			(at 186.69 116.84 0)
 			(show_name no)
