File: kicad/mission-board/expander_mux.kicad_sch (KiCad schematic)
At the start: 2 parts, among them U8 MCP23017, U9 CD74HC4067

Commit message: pcb progress
Parts:
- added J22: Limit Switch Input, Connector_JST:JST_XH_B3B-XH-A_1x03_P2.50mm_Vertical, symbol Connector:Conn_01x03_Pin
Connections:
- net GND: now also J22.2 (Pin_2)
- net HBRIDGE3_BISENSE: now reaches U9.20 (I11)
- net HBRIDGE3_AISENSE: now reaches U9.21 (I10)
- net HBRIDGE2_BISENSE: now reaches U9.22 (I9)
- net BATT_VSENSE renamed HBRIDGE2_AISENSE
- net EXP_GPIO2 renamed LIMIT_SW1
- net LIMIT_SW1: now also J22.1 (Pin_1)
- net EXP_GPIO3 renamed LIMIT_SW2
- net LIMIT_SW2: now also J22.3 (Pin_3)
Changed lines of the file:
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@@
+		)
+	)
+	(label "LIMIT_SW1"
+		(at 38.1 74.93 180)
+		(effects
+			(font
+				(size 1.27 1.27)
+			)
+			(justify right)
 		)
 	)
@@
 		)
 	)
+	(label "GND"
+		(at 214.63 90.17 0)
+		(effects
+			(font
+				(size 1.27 1.27)
+			)
+			(justify left)
+		)
+	)
 	(label "ESP_3V3"
 		(at 162.56 62.23 0)
@@
 		)
 	)
+	(label "LIMIT_SW2"
+		(at 214.63 92.71 0)
+		(effects
+			(font
+				(size 1.27 1.27)
+			)
+			(justify left)
+		)
+	)
+	(label "LIMIT_SW1"
+		(at 214.63 87.63 0)
+		(effects
+			(font
+				(size 1.27 1.27)
+			)
+			(justify left)
+		)
+	)
+	(label "LIMIT_SW2"
+		(at 38.1 77.47 180)
+		(effects
+			(font
+				(size 1.27 1.27)
+			)
+			(justify right)
+		)
+	)
 	(label "MUX_S3"
 		(at 33.02 67.31 180)
@@
 		)
 	)
-	(hierarchical_label "EXP_GPIO2"
-		(shape output)
-		(at 38.1 74.93 180)
+	(hierarchical_label "HBRIDGE2_AISENSE"
+		(shape input)
+		(at 116.84 67.31 180)
 		(effects
 			(font
@@
 		)
 	)
-	(hierarchical_label "EXP_GPIO3"
-		(shape output)
-		(at 38.1 77.47 180)
-		(effects
-			(font
-				(size 1.27 1.27)
-			)
-			(justify right)
-		)
-	)
 	(hierarchical_label "MOSFET2_GATE"
 		(shape output)
@@
 		)
 	)
+	(hierarchical_label "HBRIDGE3_AISENSE"
+		(shape input)
+		(at 162.56 69.85 0)
+		(effects
+			(font
+				(size 1.27 1.27)
+			)
+			(justify left)
+		)
+	)
 	(hierarchical_label "HBRIDGE_NFAULT"
 		(shape input)
@@
 		)
 	)
-	(hierarchical_label "BATT_VSENSE"
-		(shape input)
-		(at 116.84 67.31 180)
-		(effects
-			(font
-				(size 1.27 1.27)
-			)
-			(justify right)
+	(hierarchical_label "HBRIDGE2_BISENSE"
+		(shape input)
+		(at 162.56 67.31 0)
+		(effects
+			(font
+				(size 1.27 1.27)
+			)
+			(justify left)
 		)
 	)
@@
 			)
 			(justify right)
+		)
+	)
+	(hierarchical_label "HBRIDGE3_BISENSE"
+		(shape input)
+		(at 162.56 72.39 0)
+		(effects
+			(font
+				(size 1.27 1.27)
+			)
+			(justify left)
 		)
 	)
@@
 					(unit 1)
 				)
+			)
+		)
+	)
+	(symbol
+		(lib_id "Connector:Conn_01x03_Pin")
+		(at 209.55 90.17 0)
+		(unit 1)
+		(body_style 1)
+		(exclude_from_sim no)
+		(in_bom yes)
+		(on_board yes)
+		(in_pos_files yes)
+		(dnp no)
+		(property "Reference" "J22"
+			(at 207.01 90.932 0)
+			(show_name no)
+			(do_not_autoplace no)
+			(effects
+				(font
+					(size 1.27 1.27)
+				)
+			)
+		)
+		(property "Value" "Limit Switch Input"
+			(at 215.138 95.25 0)
+			(show_name no)
+			(do_not_autoplace no)
+			(effects
+				(font
+					(size 1.27 1.27)
+				)
+			)
+		)
+		(property "Footprint" "Connector_JST:JST_XH_B3B-XH-A_1x03_P2.50mm_Vertical"
+			(at 209.55 90.17 0)
+			(hide yes)
+			(show_name no)
+			(do_not_autoplace no)
+			(effects
+				(font
+					(size 1.27 1.27)
+				)
+			)
+		)
+		(property "Datasheet" ""
+			(at 209.55 90.17 0)
+			(hide yes)
+			(show_name no)
+			(do_not_autoplace no)
+			(effects
+				(font
+					(size 1.27 1.27)
+				)
+			)
+		)
+		(property "Description" "2x limit/position switches, active-low with MCP23017 internal pull-ups (GPB6/GPB7); pin3 shared GND return"
+			(at 209.55 90.17 0)
+			(hide yes)
+			(show_name no)
+			(do_not_autoplace no)
+			(effects
+				(font
+					(size 1.27 1.27)
+				)
+			)
+		)
+		(pin "1"
+		)
+		(pin "2"
+		)
+		(pin "3"
+		)
+		(instances
+			(project "mission-board"
+				(path "/3c2d59a7-2630-4960-9e06-c91fd9ee8058/6ee8624e-b48f-4d4c-9cbb-96fb55ac0c14"
+					(reference "J22")
+					(unit 1)
+				)

Commit message: progress on v1 of mission board
Parts:
- added C19, C20: 100nF, Capacitor_SMD:C_0402_1005Metric, symbol Device:C
- added R35, R36: 4.7k, Resistor_SMD:R_0402_1005Metric, symbol Device:R
Connections:
- net ESP_3V3: now also C19.1, C20.1, R35.1, R36.1
- net GND: now also C19.2, C20.2
- net I2C_SCL: now also R35.2
- net I2C_SDA: now also R36.2
- net LIMIT_SW2: now also U8.5 (GPB4); no longer U8.8 (GPB7)
- net SPI_CS: now also U8.8 (GPB7); no longer U8.5 (GPB4)

Commit message: Kicad FC v3.1 complete, Mission Controller and UWB boards v1 complete, firmware v2 complete!
Parts:
- J22: LCSC Part (none) -> C144394
Connections:
- net CAM_PWDN: now also U8.3 (GPB2); no longer U8.27 (GPA6)
- net EXP_ADC: now also U9.16 (I15); no longer U9.23 (I8)
- net HBRIDGE_NFAULT: now also U8.5 (GPB4); no longer U8.26 (GPA5)
- net HBRIDGE_NSLEEP: now also U8.4 (GPB3); no longer U8.25 (GPA4)
- net LIMIT_SW1: now also U8.1 (GPB0); no longer U8.7 (GPB6)
- net LIMIT_SW2: now also U8.2 (GPB1); no longer U8.5 (GPB4)
- net MOSFET1_GATE: now also U8.27 (GPA6); no longer U8.21 (GPA0)
- net MOSFET2_GATE: now also U8.26 (GPA5); no longer U8.22 (GPA1)
- net MOSFET3_GATE: now also U8.25 (GPA4); no longer U8.23 (GPA2)
- net MUX_S0: now also U8.22 (GPA1); no longer U8.1 (GPB0)
- net MUX_S1: now also U8.21 (GPA0); no longer U8.2 (GPB1)
- net MUX_S2: now also U8.23 (GPA2); no longer U8.3 (GPB2)
- net MUX_S3: now also U8.7 (GPB6); no longer U8.4 (GPB3)
- net SPI_CS: no longer names the net of U8.8 (GPB7)
- no-connect marks 10 -> 8
Changed lines of the file:
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@@
-	)
-	(no_connect
-		(at 162.56 69.85)
 	)
 	(no_connect
@@
 	)
 	(no_connect
-		(at 162.56 82.55)
+		(at 63.5 82.55)
 	)
 	(no_connect
-		(at 63.5 82.55)
-	)
-	(no_connect
-		(at 162.56 72.39)
-	)
-	(no_connect
-		(at 162.56 67.31)
+		(at 38.1 77.47)
 	)
 	(no_connect
@@
 	)
 	(no_connect
+		(at 162.56 64.77)
+	)
+	(no_connect
 		(at 162.56 74.93)
 	)
-	(wire
-		(pts
-			(xy 38.1 67.31) (xy 33.02 67.31)
-		)
-		(stroke
-			(width 0)
-			(type default)
-		)
-	)
-	(wire
-		(pts
-			(xy 38.1 62.23) (xy 33.02 62.23)
-		)
-		(stroke
-			(width 0)
-			(type default)
-		)
-	)
-	(wire
-		(pts
-			(xy 38.1 64.77) (xy 33.02 64.77)
-		)
-		(stroke
-			(width 0)
-			(type default)
-		)
-	)
-	(wire
-		(pts
-			(xy 38.1 59.69) (xy 33.02 59.69)
-		)
-		(stroke
-			(width 0)
-			(type default)
-		)
-	)
 	(label "MUX_S2"
-		(at 33.02 64.77 180)
-		(effects
-			(font
-				(size 1.27 1.27)
-			)
-			(justify right)
+		(at 63.5 72.39 0)
+		(effects
+			(font
+				(size 1.27 1.27)
+			)
+			(justify left)
 		)
 	)
 	(label "MUX_S0"
-		(at 33.02 59.69 180)
-		(effects
-			(font
-				(size 1.27 1.27)
-			)
-			(justify right)
+		(at 63.5 74.93 0)
+		(effects
+			(font
+				(size 1.27 1.27)
+			)
+			(justify left)
 		)
 	)
@@
 	)
 	(label "LIMIT_SW1"
-		(at 38.1 74.93 180)
+		(at 38.1 59.69 180)
 		(effects
 			(font
@@
 	)
 	(label "MUX_S1"
-		(at 33.02 62.23 180)
-		(effects
-			(font
-				(size 1.27 1.27)
-			)
-			(justify right)
+		(at 63.5 77.47 0)
+		(effects
+			(font
+				(size 1.27 1.27)
+			)
+			(justify left)
 		)
 	)
@@
 	)
 	(label "LIMIT_SW2"
-		(at 38.1 69.85 180)
+		(at 38.1 62.23 180)
 		(effects
 			(font
@@
 	)
 	(label "MUX_S3"
-		(at 33.02 67.31 180)
+		(at 38.1 74.93 180)
 		(effects
 			(font
@@
 	(hierarchical_label "HBRIDGE_NSLEEP"
 		(shape output)
-		(at 63.5 67.31 0)
-		(effects
-			(font
-				(size 1.27 1.27)
-			)
-			(justify left)
+		(at 38.1 67.31 180)
+		(effects
+			(font
+				(size 1.27 1.27)
+			)
+			(justify right)
 		)
 	)
@@
 	(hierarchical_label "MOSFET3_GATE"
 		(shape output)
-		(at 63.5 72.39 0)
+		(at 63.5 67.31 0)
 		(effects
 			(font
@@
 	(hierarchical_label "EXP_ADC"
 		(shape input)
-		(at 162.56 64.77 0)
+		(at 162.56 82.55 0)
 		(effects
 			(font
@@
 	(hierarchical_label "MOSFET2_GATE"
 		(shape output)
-		(at 63.5 74.93 0)
-		(effects
-			(font
-				(size 1.27 1.27)
-			)
-			(justify left)
-		)
-	)
-	(hierarchical_label "SPI_CS"
-		(shape output)
-		(at 38.1 77.47 180)
-		(effects
-			(font
-				(size 1.27 1.27)
-			)
-			(justify right)
+		(at 63.5 64.77 0)
+		(effects
+			(font
+				(size 1.27 1.27)
+			)
+			(justify left)
 		)
 	)
@@
 	(hierarchical_label "HBRIDGE_NFAULT"
 		(shape input)
-		(at 63.5 64.77 0)
-		(effects
-			(font
-				(size 1.27 1.27)
-			)
-			(justify left)
+		(at 38.1 69.85 180)
+		(effects
+			(font
+				(size 1.27 1.27)
+			)
+			(justify right)
 		)
 	)
@@
 	(hierarchical_label "CAM_PWDN"
 		(shape output)
-		(at 63.5 62.23 0)
-		(effects
-			(font
-				(size 1.27 1.27)
-			)
-			(justify left)
+		(at 38.1 64.77 180)
+		(effects
+			(font
+				(size 1.27 1.27)
+			)
+			(justify right)
 		)
 	)
@@
 	(hierarchical_label "MOSFET1_GATE"
 		(shape output)
-		(at 63.5 77.47 0)
+		(at 63.5 62.23 0)
 		(effects
 			(font
@@
 			(at 209.55 90.17 0)
 			(hide yes)
+			(show_name no)
+			(do_not_autoplace no)
+			(effects
+				(font
+					(size 1.27 1.27)
+				)
+			)
+		)
+		(property "LCSC Part" "C144394"
+			(at 209.55 90.17 0)
+			(hide yes)
