File: kicad/mission-board/mission-board.kicad_pcb (KiCad board)
At the start: 2 copper layers, 100 x 74 mm, 106 parts, among them J1 Servo 1, J10 MOSFET Ch2 Out, J11 MOSFET Ch3 Out, J12 MOSFET Ch4 Out, J13 Camera FPC, J14 I2C Expansion, J15 SPI Expansion, J16 GPIO/ADC Expansion, J17 Debug UART, J18 Inter-ESP UART, J19 Servo 5, J2 Servo 2, J20 Servo 6, J21 Fast IO Expansion, J22 Limit Switch Input, J23 H-Bridge Ch Out, J24 H-Bridge Ch Out, J25 H-Bridge Ch Out, J26 H-Bridge Ch Out, J3 Servo 3, J4 Servo 4, J5 USB-C, J6 Actuator Power In, J7 H-Bridge Ch Out, J8 H-Bridge Ch Out, J9 MOSFET Ch1 Out, Q1 reverse polarity protection, Q2 AO3400A, Q3 AO3400A, Q4 AO3400A, Q5 AO3400A, SW1 TS-1088, SW2 TS-1088, U1 INA180A2IDBVR, U10 24MHz Oscillator, U11 ESP32-S3-WROOM-1, U12 PCA9685PW, U13 DRV8833, U14 DRV8833, U2 XC6220B331PR-G, U3 DRV8833, U4 INA180A2IDBVR, U5 INA180A2IDBVR, U6 INA180A2IDBVR, U7 INA180A2IDBVR, U8 MCP23017, U9 CD74HC4067

Commit message: progress on v1 of mission board
Parts:
- removed D1, D2: ESD5Z5.0T1G, Diode_SMD:D_SOD-523
- removed MH2: MountingHole_2.2mm_M2, MountingHole_2.2mm_M2
- added C15: 4.7uF, Capacitor_SMD:C_0603_1608Metric, F.Cu at (72.3, 88.0)
- added C16: 100nF, Capacitor_SMD:C_0402_1005Metric, F.Cu at (82.8, 106.9)
- added C17: 10uF, Capacitor_SMD:C_0805_2012Metric, F.Cu at (79.7, 118.3)
- added C18: 10uF, Capacitor_SMD:C_0805_2012Metric, F.Cu at (88.7, 118.3)
- added C19: 100nF, Capacitor_SMD:C_0402_1005Metric, F.Cu at (145.2, 102.2)
- added C20: 100nF, Capacitor_SMD:C_0402_1005Metric, F.Cu at (104.2, 104.6)
- added C21: 100nF, Capacitor_SMD:C_0402_1005Metric, F.Cu at (135.6, 118.5)
- added C22: 100nF, Capacitor_SMD:C_0402_1005Metric, F.Cu at (135.6, 127.2)
- added C23: 100nF, Capacitor_SMD:C_0402_1005Metric, F.Cu at (135.6, 136.0)
- added C24: 100nF, Capacitor_SMD:C_0402_1005Metric, F.Cu at (135.6, 145.0)
- added C25: 1uF, Capacitor_SMD:C_0402_1005Metric, F.Cu at (112.0, 90.6)
- added C26: 1uF, Capacitor_SMD:C_0402_1005Metric, F.Cu at (118.4, 90.6)
- added C27: 1uF, Capacitor_SMD:C_0402_1005Metric, F.Cu at (120.0, 92.0)
- added C28: 1uF, Capacitor_SMD:C_0402_1005Metric, F.Cu at (126.0, 90.6)
- added C29: 100nF, Capacitor_SMD:C_0402_1005Metric, F.Cu at (90.4, 108.0)
- added R35: 4.7k, Resistor_SMD:R_0402_1005Metric, F.Cu at (85.0, 89.5)
- added R36: 4.7k, Resistor_SMD:R_0402_1005Metric, F.Cu at (85.0, 91.0)
- added R37: 10k, Resistor_SMD:R_0402_1005Metric, F.Cu at (114.2, 94.6)
- added R38: 10k, Resistor_SMD:R_0402_1005Metric, F.Cu at (117.0, 94.6)
- added U15: USBLC6-2SC6, Package_TO_SOT_SMD:SOT-23-6, F.Cu at (74.8, 92.9)
- added U16: XC6206P282MR, Package_TO_SOT_SMD:SOT-23-3, F.Cu at (115.2, 90.6)
- added U17: XC6206P122MR, Package_TO_SOT_SMD:SOT-23-3, F.Cu at (123.0, 90.6)
- added U18: PCA9685PW, easyeda2kicad:TSSOP-28_L9.7-W4.4-P0.65-LS6.4-TL, F.Cu at (96.5, 110.5)
- C12, C14, C5: value 470nF -> 2.2uF; footprint Capacitor_SMD:C_0402_1005Metric -> Capacitor_SMD:C_0603_1608Metric
- C7: value 100nF -> 1uF
- J6: value Actuator Power In -> Actuator Power In (5-6V BEC ONLY)
- R11, R12, R31, R32, R33, R34: value 1R -> 0.2R; footprint Resistor_SMD:R_0603_1608Metric -> Resistor_SMD:R_1206_3216Metric
- moved MH4 83.2 mm to (129.8, 145.2)
- moved R12 52.3 mm to (71.0, 113.4), turned to 90 degrees
- moved C7 49.3 mm to (68.0, 62.0)
- moved C8 48.5 mm to (74.5, 62.6), turned to 90 degrees
- moved R34 44.5 mm to (89.3, 113.4), turned to 90 degrees
- moved R11 43.8 mm to (68.5, 113.4), turned to 90 degrees
- moved R26 43.7 mm to (71.5, 62.0), turned to 0 degrees
- moved C14 42.4 mm to (86.4, 118.5), turned to 90 degrees
- moved U8 42.2 mm to (134.4, 105.6), turned to 180 degrees
- moved R33 42.0 mm to (86.8, 113.4), turned to 90 degrees
- moved C12 38.6 mm to (77.4, 118.5), turned to 90 degrees
- moved C2 37.8 mm to (73.7, 65.8), turned to 90 degrees
- moved C13 37.5 mm to (90.6, 118.7), turned to 90 degrees
- moved MH1 36.2 mm to (65.2, 79.4)
- moved C9 34.5 mm to (78.5, 71.3), turned to 90 degrees
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Connections:
- D9 pad 2: /esp32_core/LED_NODE -> /esp32_core/LED_A
- J13 pad 1: /CAM_D0 -> unconnected-(J13-Pad1)
- J13 pad 10: /CAM_VSYNC -> /GND
- J13 pad 11: /CAM_HREF -> /CAM_D6
- J13 pad 13: /I2C_SCL -> /CAM_D7
- J13 pad 14: /I2C_SDA -> /ESP_3V3
- J13 pad 15: /CAM_PWDN -> /camera/CAM_1V2
- J13 pad 16: /CAM_RESET -> /CAM_HREF
- J13 pad 17: /GND -> /CAM_PWDN
- J13 pad 18: /ESP_3V3 -> /CAM_VSYNC
- J13 pad 19: unconnected-(J13-Pad19) -> /CAM_RESET
- J13 pad 2: /CAM_D1 -> unconnected-(J13-Pad2)
- J13 pad 20: unconnected-(J13-Pad20) -> /I2C_SCL
- J13 pad 21: unconnected-(J13-Pad21) -> /camera/CAM_2V8
- J13 pad 22: unconnected-(J13-Pad22) -> /I2C_SDA
- J13 pad 23: unconnected-(J13-Pad23) -> /GND
- J13 pad 4: /CAM_D3 -> /CAM_D1
- J13 pad 5: /CAM_D4 -> /CAM_D3
- J13 pad 6: /CAM_D5 -> /CAM_D0
- J13 pad 7: /CAM_D6 -> /CAM_D4
- J13 pad 8: /CAM_D7 -> /CAM_PCLK
- J13 pad 9: /CAM_PCLK -> /CAM_D5
- J24 pad 1: /h_bridge/HBRIDGE2_BOUT1 -> /h_bridge/HBRIDGE2_BOUT2
- J24 pad 2: /h_bridge/HBRIDGE2_BOUT2 -> /h_bridge/HBRIDGE2_BOUT1
- J26 pad 1: /h_bridge/HBRIDGE3_BOUT1 -> /h_bridge/HBRIDGE3_BOUT2
- J26 pad 2: /h_bridge/HBRIDGE3_BOUT2 -> /h_bridge/HBRIDGE3_BOUT1
- J8 pad 1: /h_bridge/HBRIDGE_BOUT1 -> /h_bridge/HBRIDGE_BOUT2
- J8 pad 2: /h_bridge/HBRIDGE_BOUT2 -> /h_bridge/HBRIDGE_BOUT1
- Q1 pad 2: /power/BATT_IN -> /power/ACT_PWR_PRESHUNT
- Q1 pad 3: /power/ACT_PWR_PRESHUNT -> /power/BATT_IN
- R28 pad 2: /esp32_core/LED_NODE -> /esp32_core/LED_A
- U10 pad 1: unconnected-(U10-Tri-state-Pad1) -> /ESP_3V3
- U11 pad 10: /I2C_SDA -> /SENSE_MUX_OUT
- U11 pad 12: /CAM_D4 -> /I2C_SDA
- U11 pad 15: /INTER_ESP_UART_RX -> /esp32_core/FASTIO3
- U11 pad 17: /CAM_D5 -> /SPI_SCK
- U11 pad 18: /CAM_D6 -> /SPI_MISO
- U11 pad 19: /CAM_D7 -> /SPI_MOSI
- U11 pad 20: /HBRIDGE_AIN1 -> /INTER_ESP_UART_RX
- U11 pad 21: /HBRIDGE_AIN2 -> /INTER_ESP_UART_TX
- U11 pad 22: /HBRIDGE_BIN1 -> /CAM_D2
- U11 pad 23: /SPI_MOSI -> /CAM_D1
- U11 pad 24: /CAM_D1 -> /CAM_D3
- U11 pad 25: /CAM_D2 -> /CAM_D0
- U11 pad 26: /CAM_D0 -> /HBRIDGE_BIN2
- U11 pad 31: /SPI_MISO -> /CAM_D4
- U11 pad 32: /SPI_SCK -> /CAM_PCLK
- U11 pad 33: /CAM_PCLK -> /CAM_D5
- U11 pad 34: /CAM_VSYNC -> /CAM_D6
- U11 pad 35: /CAM_HREF -> /CAM_D7
- U11 pad 38: /CAM_D3 -> /esp32_core/FASTIO2
- U11 pad 39: /SENSE_MUX_OUT -> /esp32_core/FASTIO1
- U11 pad 4: /MCP_INT -> /HBRIDGE_AIN1
- U11 pad 5: /esp32_core/FASTIO1 -> /HBRIDGE_AIN2
- U11 pad 6: /esp32_core/FASTIO2 -> /HBRIDGE_BIN1
- U11 pad 7: /esp32_core/FASTIO3 -> /CAM_VSYNC
- U11 pad 8: /HBRIDGE_BIN2 -> /CAM_HREF
- U11 pad 9: /INTER_ESP_UART_TX -> /MCP_INT
- U12 pad 10: /servo_out/SERVO5 -> /servo_out/SERVO3
- U12 pad 12: /HBRIDGE2_AIN1 -> unconnected-(U12-LED6-Pad12)
- U12 pad 13: /HBRIDGE2_AIN2 -> unconnected-(U12-LED7-Pad13)
- U12 pad 15: /HBRIDGE2_BIN1 -> unconnected-(U12-LED8-Pad15)
- U12 pad 16: /HBRIDGE2_BIN2 -> unconnected-(U12-LED9-Pad16)
- U12 pad 17: /HBRIDGE3_AIN1 -> unconnected-(U12-LED10-Pad17)
- U12 pad 18: /HBRIDGE3_AIN2 -> unconnected-(U12-LED11-Pad18)
- U12 pad 19: /HBRIDGE3_BIN1 -> unconnected-(U12-LED12-Pad19)
- U12 pad 20: /HBRIDGE3_BIN2 -> unconnected-(U12-LED13-Pad20)
- U12 pad 7: /servo_out/SERVO2 -> /servo_out/SERVO4
- U12 pad 8: /servo_out/SERVO3 -> /servo_out/SERVO2
- U12 pad 9: /servo_out/SERVO4 -> /servo_out/SERVO5
- U8 pad 5: /SPI_CS -> /expander_mux/LIMIT_SW2
- U8 pad 8: /expander_mux/LIMIT_SW2 -> /SPI_CS
Routing:
- net /GND: track 0.00 -> 140.5 mm, vias 0 -> 93
- net /ACT_PWR: track 0.00 -> 58.5 mm
- net /I2C_SCL: track 0.00 -> 43.8 mm, vias 0 -> 3
- net /I2C_SDA: track 0.00 -> 43.1 mm, vias 0 -> 3
- net /SENSE_MUX_OUT: track 0.00 -> 34.9 mm, vias 0 -> 2
- net /h_bridge/HBRIDGE3_BOUT2: track 0.00 -> 18.0 mm
- net /h_bridge/HBRIDGE2_BOUT2: track 0.00 -> 17.9 mm
- net /h_bridge/HBRIDGE_BOUT2: track 0.00 -> 17.3 mm
- net /servo_out/SERVO1: track 0.00 -> 17.1 mm
- net /h_bridge/HBRIDGE3_BOUT1: track 0.00 -> 17.0 mm
- net /h_bridge/HBRIDGE2_BOUT1: track 0.00 -> 16.9 mm
- net /HBRIDGE_AISENSE: track 0.00 -> 16.7 mm, vias 0 -> 2
- net /h_bridge/HBRIDGE_BOUT1: track 0.00 -> 16.5 mm
- net /servo_out/SERVO4: track 0.00 -> 16.0 mm
- net /HBRIDGE_BISENSE: track 0.00 -> 15.7 mm, vias 0 -> 2
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- added copper zone on F.Cu, net /ACT_PWR
- added copper zone on B.Cu, net /GND
- added copper zone on F.Cu, net /GND

Commit message: Kicad FC v3.1 complete, Mission Controller and UWB boards v1 complete, firmware v2 complete!
Parts:
- removed J15: SPI Expansion, Connector_PinHeader_2.54mm:PinHeader_1x06_P2.54mm_Vertical
- removed Q1: reverse polarity protection, easyeda2kicad:SOT-23-3_L2.9-W1.6-P1.90-LS2.8-BR
- removed R7: 100K, Resistor_SMD:R_0402_1005Metric
- added C30: 47uF, Capacitor_SMD:C_1206_3216Metric, F.Cu at (141.6, 146.5)
- added C31: 47uF, Capacitor_SMD:C_1206_3216Metric, F.Cu at (65.7, 122.2)
- added C32: 47uF, Capacitor_SMD:C_1206_3216Metric, F.Cu at (94.6, 135.8)
- added C33: 47uF, Capacitor_SMD:C_1206_3216Metric, F.Cu at (94.6, 141.6)
- added G***: LOGO, LOGO, B.Cu at (122.8, 119.0)
- C17, C18, C3, C9: value 10uF -> 22uF
- J6: value Actuator Power In (5-6V BEC ONLY) -> Actuator Power In; footprint Connector_JST:JST_XH_B2B-XH-A_1x02_P2.50mm_Vertical -> Connector_AMASS:AMASS_XT30UPB-M_1x02_P5.0mm_Vertical
- R8: value 0.02R -> 0.005R
- moved R38 32.6 mm to (145.5, 110.4), turned to 180 degrees
- moved C7 28.0 mm to (85.4, 83.9), turned to -90 degrees
- moved R37 26.5 mm to (140.6, 97.4), turned to -90 degrees
- moved D4 23.6 mm to (76.9, 86.0), turned to -90 degrees
- moved R26 23.2 mm to (85.4, 80.5), turned to 90 degrees
- moved D3 19.4 mm to (74.1, 86.0), turned to -90 degrees
- moved C8 17.5 mm to (83.8, 77.5)
- moved C1 17.3 mm to (80.7, 83.4)
- moved U2 15.6 mm to (75.8, 80.2), turned to -90 degrees
- moved C2 13.8 mm to (80.8, 77.6), turned to 0 degrees
- moved C19 13.6 mm to (132.5, 97.3)
- moved J17 11.3 mm to (149.1, 78.5), turned to -90 degrees
- moved C9 10.4 mm to (83.2, 80.6), turned to -90 degrees
- moved SW1 8.35 mm to (66.4, 84.8), turned to 180 degrees
- moved C16 8.10 mm to (74.7, 106.2), turned to -90 degrees
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Connections:
- J16 pad 4: unconnected-(J16-Pin_4-Pad4) -> /FASTIO4
- J16 pad 5: unconnected-(J16-Pin_5-Pad5) -> /FASTIO5
- J18 pad 1: /INTER_ESP_UART_TX -> /GND
- J18 pad 3: /GND -> /INTER_ESP_UART_TX
- J6 pad 1: /power/BATT_IN -> /GND
- J6 pad 2: /GND -> /power/ACT_PWR_PRESHUNT
- U11 pad 17: /SPI_SCK -> /FASTIO4
- U11 pad 18: /SPI_MISO -> /FASTIO5
- U11 pad 19: /SPI_MOSI -> unconnected-(U11-IO11-Pad19)
- U11 pad 20: /INTER_ESP_UART_RX -> /INTER_ESP_UART_TX
- U11 pad 21: /INTER_ESP_UART_TX -> /INTER_ESP_UART_RX
- U11 pad 22: /CAM_D2 -> /CAM_D0
- U11 pad 23: /CAM_D1 -> /CAM_D3
- U11 pad 24: /CAM_D3 -> /CAM_D1
- U11 pad 25: /CAM_D0 -> /CAM_D2
- U18 pad 12: /HBRIDGE3_BIN1 -> /HBRIDGE3_BIN2
- U18 pad 13: /HBRIDGE3_BIN2 -> /HBRIDGE3_BIN1
- U18 pad 8: /HBRIDGE2_BIN1 -> /HBRIDGE2_BIN2
- U18 pad 9: /HBRIDGE2_BIN2 -> /HBRIDGE2_BIN1
- U8 pad 1: /expander_mux/MUX_S0 -> /expander_mux/LIMIT_SW1
- U8 pad 2: /expander_mux/MUX_S1 -> /expander_mux/LIMIT_SW2
- U8 pad 21: /MOSFET1_GATE -> /expander_mux/MUX_S1
- U8 pad 22: /MOSFET2_GATE -> /expander_mux/MUX_S0
- U8 pad 23: /MOSFET3_GATE -> /expander_mux/MUX_S2
- U8 pad 25: /HBRIDGE_NSLEEP -> /MOSFET3_GATE
- U8 pad 26: /HBRIDGE_NFAULT -> /MOSFET2_GATE
- U8 pad 27: /CAM_PWDN -> /MOSFET1_GATE
- U8 pad 3: /expander_mux/MUX_S2 -> /CAM_PWDN
- U8 pad 4: /expander_mux/MUX_S3 -> /HBRIDGE_NSLEEP
- U8 pad 5: /expander_mux/LIMIT_SW2 -> /HBRIDGE_NFAULT
- U8 pad 7: /expander_mux/LIMIT_SW1 -> /expander_mux/MUX_S3
- U8 pad 8: /SPI_CS -> unconnected-(U8-GPB7-Pad8)
- U9 pad 16: unconnected-(U9-I15-Pad16) -> /EXP_ADC
- U9 pad 23: /EXP_ADC -> unconnected-(U9-I8-Pad23)
Routing:
- net /I2C_SCL: track 43.8 -> 149.7 mm, vias 3 -> 6
- net /I2C_SDA: track 43.1 -> 141.2 mm, vias 3 -> 8
- net /HBRIDGE_NSLEEP: track 1.30 -> 96.6 mm, vias 2 -> 4
- net /esp32_core/FASTIO3: track 0.00 -> 87.9 mm, vias 0 -> 3
- net /HBRIDGE_NFAULT: track 2.15 -> 86.6 mm, vias 3 -> 4
- net /GND: track 140.5 -> 219.8 mm, vias 93 -> 247
- net /ESP_3V3: track 5.19 -> 82.7 mm, vias 0 -> 42
- net /FASTIO5: track 0.00 -> 77.0 mm, vias 0 -> 1
- net /FASTIO4: track 0.00 -> 76.5 mm, vias 0 -> 1
- net /MCP_INT: track 1.54 -> 71.0 mm, vias 1 -> 4
- net /esp32_core/FASTIO2: track 0.00 -> 60.0 mm, vias 0 -> 2
- net /esp32_core/FASTIO1: track 0.00 -> 58.9 mm, vias 0 -> 2
- net /EXP_ADC: track 0.00 -> 51.1 mm, vias 0 -> 3
- net /HBRIDGE_AIN1: track 1.50 -> 52.4 mm, vias 1 -> 2
- net /HBRIDGE_AISENSE: track 16.7 -> 66.5 mm, vias 2 -> 4
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- added copper zone on In2.Cu, net /ACT_PWR
- added copper zone on F.Cu, net /ESP_3V3
- added copper zone on In2.Cu, net /ESP_3V3
- added copper zone on In1.Cu, net /GND
- added copper zone on F.Cu, net /power/ACT_PWR_PRESHUNT
Other:
- outline, holes or cut-outs redrawn
- copper layers 2 -> 4
- board text added: "+ -"
- board text added: "5V"
- board text added: "BOOT"
- board text added: "EXT CONNS"
- board text added: "FC UART"
- board text added: "GND"
- board text added: "HBRIDGE OUTPUTS"
- board text added: "LIMIT SWITCHES"
- board text added: "MOSFET OUTPUTS"
- board text added: "Mission Board v1.0 TMB October 2026"
- board text added: "RST"
- board text added: "S P G"
- board text added: "SERVO OUTPUTS"
