File: kicad/mission-board/mission-board.kicad_sch (KiCad schematic)
At the start: 0 parts

Commit message: pcb progress
Other:
- sheet expander_mux ports: added HBRIDGE2_AISENSE, HBRIDGE2_BISENSE, HBRIDGE3_AISENSE, HBRIDGE3_BISENSE; removed BATT_VSENSE, EXP_GPIO2, EXP_GPIO3
- sheet expansion_io ports: added none; removed EXP_GPIO2, EXP_GPIO3
- sheet h_bridge ports: added HBRIDGE2_AIN1, HBRIDGE2_AIN2, HBRIDGE2_AISENSE, HBRIDGE2_BIN1, HBRIDGE2_BIN2, HBRIDGE2_BISENSE, HBRIDGE3_AIN1, HBRIDGE3_AIN2, HBRIDGE3_AISENSE, HBRIDGE3_BIN1, HBRIDGE3_BIN2, HBRIDGE3_BISENSE; removed none
- sheet power ports: added none; removed BATT_VSENSE
- sheet servo_out ports: added ESP_3V3, HBRIDGE2_AIN1, HBRIDGE2_AIN2, HBRIDGE2_BIN1, HBRIDGE2_BIN2, HBRIDGE3_AIN1, HBRIDGE3_AIN2, HBRIDGE3_BIN1, HBRIDGE3_BIN2, I2C_SCL, I2C_SDA; removed none

Commit message: Kicad FC v3.1 complete, Mission Controller and UWB boards v1 complete, firmware v2 complete!
Other:
- sheet esp32_core ports: added FASTIO4, FASTIO5; removed SPI_MISO, SPI_MOSI, SPI_SCK
- sheet expander_mux ports: added none; removed SPI_CS
- sheet expansion_io ports: added FASTIO4, FASTIO5; removed SPI_CS, SPI_MISO, SPI_MOSI, SPI_SCK
Changed lines of the file:
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@@
-		)
-	)
-	(label "SPI_CS"
-		(at 181.61 133.35 180)
-		(effects
-			(font
-				(size 1.27 1.27)
-			)
-			(justify right)
 		)
 	)
@@
 		)
 	)
-	(label "SPI_MISO"
-		(at 245.11 118.11 0)
-		(effects
-			(font
-				(size 1.27 1.27)
-			)
-			(justify left bottom)
-		)
-	)
 	(label "HBRIDGE_BIN2"
 		(at 205.74 38.1 180)
@@
 		)
 	)
-	(label "SPI_MOSI"
-		(at 95.25 45.72 0)
-		(effects
-			(font
-				(size 1.27 1.27)
-			)
-			(justify left bottom)
-		)
-	)
 	(label "DEBUG_UART_RX"
 		(at 31.75 33.02 180)
@@
 		)
 	)
-	(label "SPI_MOSI"
-		(at 181.61 128.27 180)
-		(effects
-			(font
-				(size 1.27 1.27)
-			)
-			(justify right)
+	(label "FASTIO5"
+		(at 82.55 69.85 270)
+		(effects
+			(font
+				(size 1.27 1.27)
+			)
+			(justify right bottom)
 		)
 	)
@@
 		)
 	)
-	(label "SPI_SCK"
-		(at 95.25 48.26 0)
-		(effects
-			(font
-				(size 1.27 1.27)
-			)
-			(justify left bottom)
-		)
-	)
-	(label "SPI_MISO"
-		(at 31.75 38.1 180)
-		(effects
-			(font
-				(size 1.27 1.27)
-			)
-			(justify right)
-		)
-	)
 	(label "MOSFET4_ISENSE"
 		(at 250.19 81.28 0)
@@
 		)
 	)
-	(label "SPI_CS"
-		(at 95.25 106.68 0)
-		(effects
-			(font
-				(size 1.27 1.27)
-			)
-			(justify left bottom)
-		)
-	)
 	(label "HBRIDGE_NFAULT"
 		(at 31.75 101.6 180)
@@
 		)
 	)
+	(label "FASTIO5"
+		(at 220.98 143.51 270)
+		(effects
+			(font
+				(size 1.27 1.27)
+			)
+			(justify right bottom)
+		)
+	)
 	(label "HBRIDGE3_BIN2"
 		(at 166.37 40.64 0)
@@
 		)
 	)
+	(label "FASTIO4"
+		(at 226.06 143.51 270)
+		(effects
+			(font
+				(size 1.27 1.27)
+			)
+			(justify right bottom)
+		)
+	)
 	(label "CAM_D0"
 		(at 31.75 48.26 180)
@@
 		)
 	)
-	(label "SPI_SCK"
-		(at 181.61 130.81 180)
-		(effects
-			(font
-				(size 1.27 1.27)
-			)
-			(justify right)
+	(label "FASTIO4"
+		(at 80.01 69.85 270)
+		(effects
+			(font
+				(size 1.27 1.27)
+			)
+			(justify right bottom)
 		)
 	)
@@
 	(sheet
 		(at 31.75 15.24)
-		(size 63.5 53.34)
+		(size 63.5 54.61)
 		(exclude_from_sim no)
 		(in_bom yes)
@@
 		)
 		(property "Sheetfile" "esp32_core.kicad_sch"
-			(at 31.75 69.08 0)
+			(at 31.75 70.612 0)
 			(show_name no)
 			(do_not_autoplace no)
@@
 			)
 		)
-		(pin "SPI_MISO" input
-			(at 31.75 38.1 180)
-			(effects
-				(font
-					(size 1.27 1.27)
-				)
-				(justify left)
-			)
-		)
 		(pin "CAM_PCLK" input
 			(at 31.75 40.64 180)
@@
 			)
 		)
-		(pin "SPI_MOSI" output
-			(at 95.25 45.72 0)
-			(effects
-				(font
-					(size 1.27 1.27)
-				)
-				(justify right)
-			)
-		)
-		(pin "SPI_SCK" output
-			(at 95.25 48.26 0)
-			(effects
-				(font
-					(size 1.27 1.27)
-				)
-				(justify right)
+		(pin "FASTIO4" bidirectional
+			(at 80.01 69.85 270)
+			(effects
+				(font
+					(size 1.27 1.27)
+				)
+				(justify left)
+			)
+		)
+		(pin "FASTIO5" bidirectional
+			(at 82.55 69.85 270)
+			(effects
+				(font
+					(size 1.27 1.27)
+				)
+				(justify left)
 			)
 		)
@@
 		)
 		(property "Sheetfile" "expander_mux.kicad_sch"
-			(at 31.75 127.5 0)
+			(at 32.512 137.668 0)
 			(show_name no)
 			(do_not_autoplace no)
@@
 		(pin "SENSE_MUX_OUT" output
 			(at 95.25 104.14 0)
-			(effects
-				(font
-					(size 1.27 1.27)
-				)
-				(justify right)
-			)
-		)
-		(pin "SPI_CS" output
-			(at 95.25 106.68 0)
 			(effects
 				(font
@@
 			)
 		)
-		(pin "SPI_MOSI" input
-			(at 181.61 128.27 180)
-			(effects
-				(font
-					(size 1.27 1.27)
-				)
-				(justify left)
-			)
-		)
-		(pin "SPI_SCK" input
-			(at 181.61 130.81 180)
-			(effects
-				(font
-					(size 1.27 1.27)
-				)
-				(justify left)
-			)
-		)
-		(pin "SPI_CS" input
-			(at 181.61 133.35 180)
-			(effects
-				(font
-					(size 1.27 1.27)
-				)
-				(justify left)
-			)
-		)
 		(pin "EXP_GPIO1" input
 			(at 181.61 135.89 180)
@@
 			)
 		)
-		(pin "SPI_MISO" output
-			(at 245.11 118.11 0)
-			(effects
-				(font
-					(size 1.27 1.27)
-				)
-				(justify right)
-			)
-		)
 		(pin "EXP_ADC" output
 			(at 245.11 120.65 0)
@@
 			)
 		)
+		(pin "FASTIO4" bidirectional
+			(at 226.06 143.51 270)
+			(effects
+				(font
+					(size 1.27 1.27)
+				)
+				(justify left)
+			)
+		)
+		(pin "FASTIO5" bidirectional
+			(at 220.98 143.51 270)
+			(effects
+				(font
+					(size 1.27 1.27)
+				)
+				(justify left)
+			)
+		)
