File: kicad/mission-board/mosfet_bank.kicad_sch (KiCad schematic)
At the start: 28 parts, among them J10 MOSFET Ch2 Out, J11 MOSFET Ch3 Out, J12 MOSFET Ch4 Out, J9 MOSFET Ch1 Out, Q2 AO3400A, Q3 AO3400A, Q4 AO3400A, Q5 AO3400A, U4 INA180A2IDBVR, U5 INA180A2IDBVR, U6 INA180A2IDBVR, U7 INA180A2IDBVR

Commit message: pcb progress
Parts:
- J10, J11, J12, J9: footprint TerminalBlock_CUI:TerminalBlock_CUI_TB007-508-02_1x02_P5.08mm_Horizontal -> Connector_JST:JST_XH_B2B-XH-A_1x02_P2.50mm_Vertical
Other:
- moved on the sheet: U4, U5, U6, U7

Commit message: progress on v1 of mission board
Parts:
- added C21, C22, C23, C24: 100nF, Capacitor_SMD:C_0402_1005Metric, symbol Device:C
Connections:
- net ESP_3V3: now also C21.1, C22.1, C23.1, C24.1
- net GND: now also C21.2, C22.2, C23.2, C24.2

Commit message: Kicad FC v3.1 complete, Mission Controller and UWB boards v1 complete, firmware v2 complete!
Parts:
- J10, J11, J12, J9: LCSC Part (none) -> C158012
Changed lines of the file:
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@@
+			)
+		)
+		(property "LCSC Part" "C158012"
+			(at 152.4 50.8 0)
+			(hide yes)
+			(show_name no)
+			(do_not_autoplace no)
+			(effects
+				(font
+					(size 1.27 1.27)
+				)
 			)
 		)
@@
 			)
 		)
+		(property "LCSC Part" "C158012"
+			(at 203.2 50.8 0)
+			(hide yes)
+			(show_name no)
+			(do_not_autoplace no)
+			(effects
+				(font
+					(size 1.27 1.27)
+				)
+			)
+		)
 		(pin "1"
 		)
@@
 			)
 		)
+		(property "LCSC Part" "C158012"
+			(at 101.6 50.8 0)
+			(hide yes)
+			(show_name no)
+			(do_not_autoplace no)
+			(effects
+				(font
+					(size 1.27 1.27)
+				)
+			)
+		)
 		(pin "1"
 		)
@@
 			(at 50.8 50.8 0)
 			(hide yes)
+			(show_name no)
+			(do_not_autoplace no)
+			(effects
+				(font
+					(size 1.27 1.27)
+				)
+			)
+		)
+		(property "LCSC Part" "C158012"
+			(at 50.8 50.8 0)
+			(hide yes)
