File: kicad/mission-board/power.kicad_sch (KiCad schematic)
At the start: 17 parts, among them J5 USB-C, J6 Actuator Power In, Q1 reverse polarity protection, U1 INA180A2IDBVR, U2 XC6220B331PR-G

Commit message: pcb progress
Parts:
- removed R10: 10K, Resistor_SMD:R_0402_1005Metric, symbol Device:R
- removed R9: 100K, Resistor_SMD:R_0402_1005Metric, symbol Device:R
Other:
- moved on the sheet: D1, D2, D3, J6, R6, R7, R8

Commit message: progress on v1 of mission board
Parts:
- removed D1, D2: ESD5Z5.0T1G, Diode_SMD:D_SOD-523, symbol Device:D_TVS
- added C15: 4.7uF, Capacitor_SMD:C_0603_1608Metric, symbol Device:C
- added C16: 100nF, Capacitor_SMD:C_0402_1005Metric, symbol Device:C
- added U15: USBLC6-2SC6, Package_TO_SOT_SMD:SOT-23-6, symbol Power_Protection:USBLC6-2SC6
- J6: value Actuator Power In -> Actuator Power In (5-6V BEC ONLY)
Connections:
- net ACT_PWR_PRESHUNT: now also Q1.2 (S); no longer Q1.3 (D)
- net BATT_IN: now also Q1.3 (D); no longer Q1.2 (S)
- net ESP_3V3: now also C16.1
- net GND: now also C15.2, C16.2, U15.2 (GND)
- net USB_DM: now also U15.3 (I/O2), U15.4 (I/O2)
- net USB_DP: now also U15.1 (I/O1), U15.6 (I/O1)
- net USB_VBUS: now also C15.1, U15.5 (VBUS)

Commit message: Kicad FC v3.1 complete, Mission Controller and UWB boards v1 complete, firmware v2 complete!
Parts:
- removed Q1: reverse polarity protection, easyeda2kicad:SOT-23-3_L2.9-W1.6-P1.90-LS2.8-BR, symbol easyeda2kicad:AO3407A
- removed R7: 100K, Resistor_SMD:R_0402_1005Metric, symbol Device:R
- added C30, C31, C32, C33: 47uF, Capacitor_SMD:C_1206_3216Metric, symbol Device:C
- C1, C2: LCSC Part C1691 -> C19702
- J6: value Actuator Power In (5-6V BEC ONLY) -> Actuator Power In; footprint Connector_JST:JST_XH_B2B-XH-A_1x02_P2.50mm_Vertical -> Connector_AMASS:AMASS_XT30UPB-M_1x02_P5.0mm_Vertical; LCSC Part (none) -> C428721
- R8: value 0.02R -> 0.005R; LCSC Part C105360 -> C393074
Connections:
- net BATT_IN is gone; now on net GND: J6.1 (Pin_1)
- net ACT_PWR: now also C30.1, C31.1, C32.1, C33.1
- net ACT_PWR_PRESHUNT: now also J6.2 (Pin_2)
- net GND: now also C30.2, C31.2, C32.2, C33.2; no longer J6.2 (Pin_2)
