File: kicad/mission-board/servo_out.kicad_sch (KiCad schematic)
At the start: 13 parts, among them J1 Servo 1, J19 Servo 5, J2 Servo 2, J20 Servo 6, J3 Servo 3, J4 Servo 4, U12 PCA9685PW

Commit message: pcb progress
Parts:
- added C10: 100nF, Capacitor_SMD:C_0402_1005Metric, symbol Device:C
Connections:
- net GND: now also U12.1 (A0), U12.14 (VSS), U12.2 (A1), U12.23 (~{OE}), U12.24 (A5), U12.25 (EXTCLK), U12.3 (A2), U12.4 (A3), U12.5 (A4), C10.2
- net SERVO1: now also U12.6 (LED0)
- net SERVO2: now also U12.7 (LED1)
- net SERVO3: now also U12.8 (LED2)
- net SERVO4: now also U12.9 (LED3)
- net SERVO5: now also U12.10 (LED4)
- net SERVO6: now also U12.11 (LED5)
- net HBRIDGE2_AIN1: now reaches U12.12 (LED6)
- net HBRIDGE2_AIN2: now reaches U12.13 (LED7)
- net HBRIDGE2_BIN1: now reaches U12.15 (LED8)
- net HBRIDGE2_BIN2: now reaches U12.16 (LED9)
- net HBRIDGE3_AIN1: now reaches U12.17 (LED10)
- net HBRIDGE3_AIN2: now reaches U12.18 (LED11)
- net HBRIDGE3_BIN1: now reaches U12.19 (LED12)
- net HBRIDGE3_BIN2: now reaches U12.20 (LED13)
- net I2C_SCL: now reaches U12.26 (SCL)
- net I2C_SDA: now reaches U12.27 (SDA)
- net ESP_3V3: now reaches U12.28 (VDD)
- net ESP_3V3: now also C10.1

Commit message: progress on v1 of mission board
Parts:
- added C29: 100nF, Capacitor_SMD:C_0402_1005Metric, symbol Device:C
- added U18: PCA9685PW, easyeda2kicad:TSSOP-28_L9.7-W4.4-P0.65-LS6.4-TL, symbol easyeda2kicad:PCA9685PW,118
Connections:
- net ESP_3V3: now also C29.1, U18.1 (A0), U18.28 (VDD)
- net GND: now also C29.2, U18.14 (VSS), U18.2 (A1), U18.23 (~{OE}), U18.24 (A5), U18.25 (EXTCLK), U18.3 (A2), U18.4 (A3), U18.5 (A4)
- net HBRIDGE2_AIN1: now also U18.6 (LED0); no longer U12.12 (LED6)
- net HBRIDGE2_AIN2: now also U18.7 (LED1); no longer U12.13 (LED7)
- net HBRIDGE2_BIN1: now also U18.8 (LED2); no longer U12.15 (LED8)
- net HBRIDGE2_BIN2: now also U18.9 (LED3); no longer U12.16 (LED9)
- net HBRIDGE3_AIN1: now also U18.10 (LED4); no longer U12.17 (LED10)
- net HBRIDGE3_AIN2: now also U18.11 (LED5); no longer U12.18 (LED11)
- net HBRIDGE3_BIN1: now also U18.12 (LED6); no longer U12.19 (LED12)
- net HBRIDGE3_BIN2: now also U18.13 (LED7); no longer U12.20 (LED13)
- net I2C_SCL: now also U18.26 (SCL)
- net I2C_SDA: now also U18.27 (SDA)
- net SERVO2: now also U12.8 (LED2); no longer U12.7 (LED1)
- net SERVO3: now also U12.10 (LED4); no longer U12.8 (LED2)
- net SERVO4: now also U12.7 (LED1); no longer U12.9 (LED3)
- net SERVO5: now also U12.9 (LED3); no longer U12.10 (LED4)
- no-connect marks 0 -> 18
Other:
- moved on the sheet: C10

Commit message: Kicad FC v3.1 complete, Mission Controller and UWB boards v1 complete, firmware v2 complete!
Parts:
- C10: LCSC Part (none) -> C1525
Connections:
- net HBRIDGE2_BIN1: now also U18.9 (LED3); no longer U18.8 (LED2)
- net HBRIDGE2_BIN2: now also U18.8 (LED2); no longer U18.9 (LED3)
- net HBRIDGE3_BIN1: now also U18.13 (LED7); no longer U18.12 (LED6)
- net HBRIDGE3_BIN2: now also U18.12 (LED6); no longer U18.13 (LED7)
Changed lines of the file:
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@@
 	(hierarchical_label "HBRIDGE3_BIN2"
 		(shape output)
-		(at 218.44 73.66 180)
+		(at 218.44 71.12 180)
 		(effects
 			(font
@@
 	(hierarchical_label "HBRIDGE3_BIN1"
 		(shape output)
-		(at 218.44 71.12 180)
+		(at 218.44 73.66 180)
 		(effects
 			(font
@@
 	(hierarchical_label "HBRIDGE2_BIN2"
 		(shape output)
-		(at 218.44 63.5 180)
+		(at 218.44 60.96 180)
 		(effects
 			(font
@@
 	(hierarchical_label "HBRIDGE2_BIN1"
 		(shape output)
-		(at 218.44 60.96 180)
+		(at 218.44 63.5 180)
 		(effects
 			(font
@@
 			)
 		)
+		(property "LCSC Part" "C1525"
+			(at 179.07 69.85 0)
+			(hide yes)
+			(show_name no)
+			(do_not_autoplace no)
+			(effects
+				(font
+					(size 1.27 1.27)
+				)
+			)
+		)
 		(pin "1"
 		)
@@
 		(dnp no)
 		(property "Reference" "U18"
-			(at 233.68 58.42 0)
+			(at 229.362 45.72 0)
 			(show_name no)
 			(do_not_autoplace no)
@@
 		)
 		(property "Value" "PCA9685PW"
-			(at 233.68 60.96 0)
-			(show_name no)
-			(do_not_autoplace no)
+			(at 225.298 42.418 0)
+			(show_name no)
+			(do_not_autoplace no)
