File: kicad/uwb-radio-kicad/uwb-radio/uwb-radio.kicad_pcb (KiCad board)
At the start: 2 copper layers, 21.5 x 27.5 mm, 5 parts, among them CN1 BM07B-GHS-TBT, M2 MountingHole_2.2mm_M2, U1 DWM3000TR13

Commit message: Kicad FC v3.1 complete, Mission Controller and UWB boards v1 complete, firmware v2 complete!
Parts:
- added C1: 22uF, Capacitor_SMD:C_0805_2012Metric_Pad1.18x1.45mm_HandSolder, F.Cu at (148.4, 91.6)
- added C2: 10uF, Capacitor_SMD:C_0805_2012Metric_Pad1.18x1.45mm_HandSolder, F.Cu at (143.6, 83.6)
- added R2: 33R, Resistor_SMD:R_0603_1608Metric_Pad0.98x0.95mm_HandSolder, F.Cu at (154.4, 92.6)
- added U2: XC6220B331PR-G, easyeda2kicad:SOT-89-5_L4.5-W2.5-P1.50-LS4.4-BR, F.Cu at (145.1, 88.0)
- H1: renamed from REF**; value MountingHole_2.2mm_M2 -> MountingHole_M2
- H2: renamed from M2; value MountingHole_2.2mm_M2 -> MountingHole_M2
- moved CN1 4.15 mm to (155.6, 88.3)
Connections:
- CN1 pad 1: +3V3 -> +5V
- U1 pad 19: /MISO -> Net-(U1-SPIMISO)
Routing:
- net Net-(U1-SPIMISO): track 0.00 -> 23.2 mm, vias 0 -> 2
- net /MISO: track 23.1 -> 1.77 mm, vias 2 -> 0
- net +5V: track 0.00 -> 15.5 mm
- net GND: track 15.0 -> 24.0 mm, vias 13 -> 18
- net /CS: track 19.9 -> 11.3 mm
- net +3V3: track 27.1 -> 20.0 mm
- net /MOSI: track 26.8 -> 20.1 mm, vias 0 -> 2
- net /INT: track 29.1 -> 25.0 mm
- net /SCK: track 24.5 -> 22.0 mm
Other:
- board text added: "M2"
- board text removed: "1 7"
