File: kicad/uwb-radio-kicad/uwb-radio/uwb-radio.kicad_sch (KiCad schematic)
At the start: 3 parts, among them CN1 BM07B-GHS-TBT, U1 DWM3000TR13

Commit message: Kicad FC v3.1 complete, Mission Controller and UWB boards v1 complete, firmware v2 complete!
Parts:
- added C1: 22uF, Capacitor_SMD:C_0805_2012Metric_Pad1.18x1.45mm_HandSolder, symbol Device:C
- added C2: 10uF, Capacitor_SMD:C_0805_2012Metric_Pad1.18x1.45mm_HandSolder, symbol Device:C
- added H1, H2: MountingHole_M2, MountingHole:MountingHole_2.2mm_M2, symbol Mechanical:MountingHole
- added R2: 33R, Resistor_SMD:R_0603_1608Metric_Pad0.98x0.95mm_HandSolder, symbol Device:R
- added U2: XC6220B331PR-G, easyeda2kicad:SOT-89-5_L4.5-W2.5-P1.50-LS4.4-BR, symbol easyeda2kicad:XC6220B331PR-G
Connections:
- net +3V3: now also C2.1, U2.5 (VOUT); no longer CN1.1
- net GND: now also C1.2, C2.2, U2.2 (VSS)
- net MISO: now also R2.2; no longer U1.19 (SPIMISO)
- new net: R2.1, U1.19 (SPIMISO)
- new net +5V: C1.1, CN1.1, U2.1 (CE), U2.4 (VIN)
- no-connect marks 10 -> 11
Other:
- moved on the sheet: R1
